Commit message: fix urdf

File: third_robot_description/urdf/third_robot.urdf (robot description, URDF)
Before this commit: robot origins, 9 links, 8 joints
Links:
- removed link front_top_lrf
- added link front_top_3durg; visual mesh filename=package://third_robot_description/meshes/3DURG/hokuyo3durg.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
Joints:
- removed joint base_to_front_top_lrf
- added joint base_to_front_top_3durg: type fixed, parent base_link, child front_top_3durg, origin xyz=0.40 0 0.75 rpy=3.14159 0 0, axis 0 1 0
