Commit message: [WIP] SteerBotからgazeboに指令値送るの成功．SetVelocity()使えない．

File: third_robot_description/urdf/third_robot_macro.xacro (robot description, xacro)
@@ -73,5 +73,5 @@
             </inertial>
         </link>
-        <joint name="base_to_steer_${right_left}" type="continuous">
+        <joint name="base_to_${right_left}_front_steer" type="continuous">
             <axis xyz="0 0 1"/>
             <parent link="base_link"/>

Commit message: [modify] yamlファイル構成を修正．yaml内でwheel_hが無い時にTFから自動計算するよう修正

File: third_robot_description/urdf/third_robot_macro.xacro (robot description, xacro)
@@ -102,5 +102,5 @@
             <child link="${right_left}_front_wheel"/>
             <!-- <origin xyz="${base_center_x+length_from_base_center_to_wheel_x} ${-reflect_right_left*length_from_base_to_wheel_y} ${radius_wheel}"/> -->
-            <origin xyz="0 0 -0.15"/>
+            <origin xyz="0 0 -0.16"/>
         </joint>
         <transmission name="tran_${right_left}_front">
