Commit message: [modify] デバッグ実行できるようファイルを修正

File: third_robot_description/urdf/third_robot.xacro (robot description, xacro)
@@ -51,4 +51,18 @@
         </visual>
     </link>
+    <link name="steer">
+        <visual>
+            <origin rpy="0 0 0" xyz="0 0 0"/>
+            <geometry>
+                <mesh filename="package://third_robot_description/meshes/LRF/UTM-30LX.dae"/>
+            </geometry>
+        </visual>
+    </link>
+    <joint name="base_to_steer" type="fixed">
+        <axis xyz="0 1 0"/>
+        <parent link="base_link"/>
+        <child link="steer"/>
+        <origin xyz="0.41 0 0.14"/>
+    </joint>
     <joint name="base_to_front_bottom_lrf" type="fixed">
         <axis xyz="0 1 0"/>

Commit message: [WIP] URDFモデルに仮想jointを付けた

File: third_robot_description/urdf/third_robot.xacro (robot description, xacro)
@@ -43,4 +43,5 @@
         <origin rpy="0 0.53 0" xyz="0.40 0 0.75"/>
     </joint>
+    <!-- front_bottom_lrf -->
     <link name="front_bottom_lrf">
         <visual>
@@ -51,4 +52,11 @@
         </visual>
     </link>
+    <joint name="base_to_front_bottom_lrf" type="fixed">
+        <axis xyz="0 1 0"/>
+        <parent link="base_link"/>
+        <child link="front_bottom_lrf"/>
+        <origin xyz="0.50 0 0.39"/>
+    </joint>
+    <!-- steer -->
     <link name="steer">
         <visual>
@@ -65,10 +73,47 @@
         <origin xyz="0.41 0 0.14"/>
     </joint>
-    <joint name="base_to_front_bottom_lrf" type="fixed">
-        <axis xyz="0 1 0"/>
+    <!-- steer_right -->
+    <link name="steer_right">
+        <visual>
+            <origin rpy="0 0 0" xyz="0 0 0"/>
+            <geometry>
+                <mesh filename="package://third_robot_description/meshes/LRF/UTM-30LX.dae"/>
+            </geometry>
+        </visual>
+        <inertial>
+            <mass value="1.0" />
+            <inertia ixx="1.0" ixy="0.0" ixz="0.0"
+                iyy="1.0" iyz="0.0"
+                izz="1.0" />
+        </inertial>
+    </link>
+    <joint name="base_to_steer_right" type="continuous">
+        <axis xyz="0 0 1"/>
         <parent link="base_link"/>
-        <child link="front_bottom_lrf"/>
-        <origin xyz="0.50 0 0.39"/>
+        <child link="steer_right"/>
+        <origin xyz="0.41 -0.25 0.34"/>
     </joint>
+    <!-- steer_left -->
+    <link name="steer_left">
+        <visual>
+            <origin rpy="0 0 0" xyz="0 0 0"/>
+            <geometry>
+                <mesh filename="package://third_robot_description/meshes/LRF/UTM-30LX.dae"/>
+            </geometry>
+        </visual>
+        <inertial>
+            <mass value="1.0" />
+            <inertia ixx="1.0" ixy="0.0" ixz="0.0"
+                iyy="1.0" iyz="0.0"
+                izz="1.0" />
+        </inertial>
+    </link>
+    <joint name="base_to_steer_left" type="continuous">
+        <axis xyz="0 0 1"/>
+        <parent link="base_link"/>
+        <child link="steer_left"/>
+        <origin xyz="0.41 0.25 0.34"/>
+    </joint>
+    <!-- rear_bottom_lrf -->
     <link name="rear_bottom_lrf">
         <visual>

Commit message: [add] xacroモデルで前wheelに仮想steerを設置

File: third_robot_description/urdf/third_robot.xacro (robot description, xacro)
@@ -24,6 +24,6 @@
     </link>
     <!-- wheels -->
-    <xacro:wheel right_left="right" reflect_right_left="1" front_rear="front" reflect_front_rear="1"/>
-    <xacro:wheel right_left="left" reflect_right_left="-1" front_rear="front" reflect_front_rear="1"/>
+    <xacro:front_wheel right_left="right" reflect_right_left="1"/>
+    <xacro:front_wheel right_left="left" reflect_right_left="-1"/>
     <xacro:wheel right_left="right" reflect_right_left="1" front_rear="rear" reflect_front_rear="-1"/>
     <xacro:wheel right_left="left" reflect_right_left="-1" front_rear="rear" reflect_front_rear="-1"/>
@@ -73,26 +73,6 @@
         <origin xyz="0.41 0 0.14"/>
     </joint>
-    <!-- steer_right -->
-    <link name="steer_right">
-        <visual>
-            <origin rpy="0 0 0" xyz="0 0 0"/>
-            <geometry>
-                <mesh filename="package://third_robot_description/meshes/LRF/UTM-30LX.dae"/>
-            </geometry>
-        </visual>
-        <inertial>
-            <mass value="1.0" />
-            <inertia ixx="1.0" ixy="0.0" ixz="0.0"
-                iyy="1.0" iyz="0.0"
-                izz="1.0" />
-        </inertial>
-    </link>
-    <joint name="base_to_steer_right" type="continuous">
-        <axis xyz="0 0 1"/>
-        <parent link="base_link"/>
-        <child link="steer_right"/>
-        <origin xyz="0.41 -0.25 0.34"/>
-    </joint>
     <!-- steer_left -->
+    <!--
     <link name="steer_left">
         <visual>
@@ -115,4 +95,5 @@
         <origin xyz="0.41 0.25 0.34"/>
     </joint>
+    -->
     <!-- rear_bottom_lrf -->
     <link name="rear_bottom_lrf">

File: third_robot_description/urdf/third_robot_macro.xacro (robot description, xacro)
@@ -56,3 +56,62 @@
         </transmission>
     </xacro:macro>
+    <!-- front wheel macro -->
+    <xacro:macro name="front_wheel" params="right_left reflect_right_left">
+        <!-- steer_right -->
+        <link name="steer_${right_left}">
+            <visual>
+                <origin rpy="0 0 0" xyz="0 0 0"/>
+                <geometry>
+                    <mesh filename="package://third_robot_description/meshes/LRF/UTM-30LX.dae"/>
+                </geometry>
+            </visual>
+            <inertial>
+                <mass value="1.0" />
+                <inertia ixx="1.0" ixy="0.0" ixz="0.0"
+                    iyy="1.0" iyz="0.0"
+                    izz="1.0" />
+            </inertial>
+        </link>
+        <joint name="base_to_steer_${right_left}" type="continuous">
+            <axis xyz="0 0 1"/>
+            <parent link="base_link"/>
+            <child link="steer_${right_left}"/>
+        <origin xyz="${base_center_x+length_from_base_center_to_wheel_x} ${-reflect_right_left*length_from_base_to_wheel_y} 0.30"/>
+        </joint>
+        <link name="${right_left}_front_wheel">
+            <visual>
+                <!-- when reflect_right_left = 1 to be 0 reflect_right_left= -1 to be PI -->
+                <origin rpy="${PI/2-reflect_right_left*PI/2} 0 0" xyz="0 0 0"/>
+                <!-- <origin rpy="${PI/2-reflect_right_left*PI/2} 0 0" xyz="0 0 0"/> -->
+                <geometry>
+                    <mesh filename="package://third_robot_description/meshes/third_robot/third_robot_wheel.dae"/>
+                </geometry>
+                ->
+            </visual>
+            <collision>
+                <origin rpy="${PI/2} 0 0" xyz="0 0 0"/>
+                <geometry>
+                    <cylinder length="${length_wheel}" radius="${radius_wheel}"/>
+                </geometry>
+            </collision>
+            <xacro:default_inertial mass="1"/>
+        </link>
+        <joint name="base_to_${right_left}_front_wheel" type="continuous">
+            <axis xyz="0 1 0"/>
+            <parent link="steer_${right_left}"/>
+            <child link="${right_left}_front_wheel"/>
+            <!-- <origin xyz="${base_center_x+length_from_base_center_to_wheel_x} ${-reflect_right_left*length_from_base_to_wheel_y} ${radius_wheel}"/> -->
+            <origin xyz="0 0 -0.15"/>
+        </joint>
+        <transmission name="tran_${right_left}_front">
+            <type>transmission_interface/SimpleTransmission</type>
+            <joint name="base_to_${right_left}_front_wheel">
+                <hardwareInterface>VelocityJointInterface</hardwareInterface>
+            </joint>
+            <actuator name="${right_left}_front">
+                <hardwareInterface>VelocityJointInterface</hardwareInterface>
+                <mechanicalReduction>1</mechanicalReduction>
+            </actuator>
+        </transmission>
+    </xacro:macro>
 </robot>

Commit message: changed 2d lidar to 3d lidar

File: third_robot_description/urdf/third_robot.xacro (robot description, xacro)
@@ -9,17 +9,17 @@
     <xacro:include filename="$(find third_robot_description)/urdf/third_robot_macro.xacro" />
     <link name="base_link">
-        <visual>
-            <origin rpy="0 0 0" xyz="0 0 0.55" />
-            <geometry>
-                <mesh filename="package://third_robot_description/meshes/third_robot/third_robot_body.dae"/>
-            </geometry>
-        </visual>
-        <collision>
-            <origin rpy="0 0 0" xyz="0 0 0.35" />
-            <geometry>
-                <box size="1.0 0.55 0.4"/>
-            </geometry>
-        </collision>
-        <xacro:default_inertial mass="10"/>
+      <visual>
+        <origin rpy="0 0 0" xyz="0 0 0.55" />
+        <geometry>
+          <mesh filename="package://third_robot_description/meshes/third_robot/third_robot_body.dae"/>
+        </geometry>
+      </visual>
+      <collision>
+        <origin rpy="0 0 0" xyz="0 0 0.35" />
+        <geometry>
+          <box size="1.0 0.55 0.4"/>
+        </geometry>
+      </collision>
+      <xacro:default_inertial mass="10"/>
     </link>
     <!-- wheels -->
@@ -29,25 +29,40 @@
     <xacro:wheel right_left="left" reflect_right_left="-1" front_rear="rear" reflect_front_rear="-1"/>
     <!-- lrf -->
-    <link name="front_top_lrf">
-        <visual>
-            <origin rpy="0 0.5 0" xyz="0 0 0"/>
-            <geometry>
-                <mesh filename="package://third_robot_description/meshes/LRF/UTM-30LX.dae"/>
-            </geometry>
-        </visual>
+    <!-- <link name="front_top_lrf"> -->
+    <!--     <visual> -->
+    <!--         <origin rpy="0 0.5 0" xyz="0 0 0"/> -->
+    <!--         <geometry> -->
+    <!--             <mesh filename="package://third_robot_description/meshes/LRF/UTM-30LX.dae"/> -->
+    <!--         </geometry> -->
+    <!--     </visual> -->
+    <!-- </link> -->
+    <!-- <joint name="base_to_front_top_lrf" type="fixed"> -->
+    <!--     <axis xyz="0 1 0"/> -->
+    <!--     <parent link="base_link"/> -->
+    <!--     <child link="front_top_lrf"/> -->
+    <!--     <origin rpy="0 0.53 0" xyz="0.40 0 0.75"/> -->
+    <!-- </joint> -->
+    <!-- lrf -->
+    <link name="front_top_3durg">
+      <visual>
+        <origin rpy="0 0 0" xyz="0 0 0"/>
+        <geometry>
+          <mesh filename="package://third_robot_description/meshes/3DURG/hokuyo3durg.dae"/>
+        </geometry>
+      </visual>
     </link>
-    <joint name="base_to_front_top_lrf" type="fixed">
-        <axis xyz="0 1 0"/>
-        <parent link="base_link"/>
-        <child link="front_top_lrf"/>
-        <origin rpy="0 0.53 0" xyz="0.40 0 0.75"/>
+    <joint name="base_to_front_top_3durg" type="fixed">
+      <axis xyz="0 1 0"/>
+      <parent link="base_link"/>
+      <child link="front_top_3durg"/>
+      <origin rpy="3.14159 0 0" xyz="0.40 0 0.75"/>
     </joint>
     <link name="front_bottom_lrf">
-        <visual>
-            <origin rpy="0 0 0" xyz="0 0 0"/>
-            <geometry>
-                <mesh filename="package://third_robot_description/meshes/LRF/UTM-30LX.dae"/>
-            </geometry>
-        </visual>
+      <visual>
+        <origin rpy="0 0 0" xyz="0 0 0"/>
+        <geometry>
+          <mesh filename="package://third_robot_description/meshes/LRF/UTM-30LX.dae"/>
+        </geometry>
+      </visual>
     </link>
     <joint name="base_to_front_bottom_lrf" type="fixed">
@@ -58,63 +73,63 @@
     </joint>
     <link name="rear_bottom_lrf">
-        <visual>
-            <origin rpy="0 0 ${PI}" xyz="0 0 0"/>
-            <geometry>
-                <mesh filename="package://third_robot_description/meshes/LRF/UTM-30LX.dae"/>
-            </geometry>
-        </visual>
+      <visual>
+        <origin rpy="0 0 ${PI}" xyz="0 0 0"/>
+        <geometry>
+          <mesh filename="package://third_robot_description/meshes/LRF/UTM-30LX.dae"/>
+        </geometry>
+      </visual>
     </link>
     <joint name="base_to_rear_bottom_lrf" type="fixed">
-        <axis xyz="0 1 0"/>
-        <parent link="base_link"/>
-        <child link="rear_bottom_lrf"/>
-        <origin  rpy="0 0 ${PI}" xyz="-0.45 0 0.35"/>
+      <axis xyz="0 1 0"/>
+      <parent link="base_link"/>
+      <child link="rear_bottom_lrf"/>
+      <origin  rpy="0 0 ${PI}" xyz="-0.45 0 0.35"/>
     </joint>
     <!-- Camera -->
     <link name="camera_link">
-        <collision>
-            <origin xyz="0 0 0" rpy="0 0 0"/>
-            <geometry>
-                <box size="${camera_link/3} ${camera_link} ${camera_link/2}"/>
-            </geometry>
-        </collision>
-        <visual>
-            <origin xyz="0 0 0" rpy="0 0 0"/>
-            <geometry>
-                <box size="${camera_link/3} ${camera_link} ${camera_link/2}"/>
-            </geometry>
-            <material name="black"/>
-        </visual>
-        <inertial>
-            <mass value="1e-5" />
-            <origin xyz="0 0 0" rpy="0 0 0"/>
-            <inertia ixx="1e-6" ixy="0" ixz="0" iyy="1e-6" iyz="0" izz="1e-6" />
-        </inertial>
+      <collision>
+        <origin xyz="0 0 0" rpy="0 0 0"/>
+        <geometry>
+          <box size="${camera_link/3} ${camera_link} ${camera_link/2}"/>
+        </geometry>
+      </collision>
+      <visual>
+        <origin xyz="0 0 0" rpy="0 0 0"/>
+        <geometry>
+          <box size="${camera_link/3} ${camera_link} ${camera_link/2}"/>
+        </geometry>
+        <material name="black"/>
+      </visual>
+      <inertial>
+        <mass value="1e-5" />
+        <origin xyz="0 0 0" rpy="0 0 0"/>
+        <inertia ixx="1e-6" ixy="0" ixz="0" iyy="1e-6" iyz="0" izz="1e-6" />
+      </inertial>
     </link>
     <joint name="base_to_camera" type="fixed">
-        <axis xyz="0 1 0" />
-        <parent link="base_link"/>
-        <child link="camera_link"/>
-        <origin rpy="0 0 0" xyz="0.45 0 0.72"/>
+      <axis xyz="0 1 0" />
+      <parent link="base_link"/>
+      <child link="camera_link"/>
+      <origin rpy="0 0 0" xyz="0.45 0 0.72"/>
     </joint>
     <transmission name="tran1">
-        <type>transmission_interface/SimpleTransmission</type>
+      <type>transmission_interface/SimpleTransmission</type>
         <joint name="base_to_left_rear_wheel">
-            <hardwareInterface>EffortJointInterface</hardwareInterface>
+          <hardwareInterface>EffortJointInterface</hardwareInterface>
         </joint>
         <actuator name="motor1">
-            <hardwareInterface>EffortJointInterface</hardwareInterface>
-            <mechanicalReduction>1</mechanicalReduction>
+          <hardwareInterface>EffortJointInterface</hardwareInterface>
+          <mechanicalReduction>1</mechanicalReduction>
         </actuator>
     </transmission>
     <transmission name="tran2">
-        <type>transmission_interface/SimpleTransmission</type>
-        <joint name="base_to_right_rear_wheel">
-            <hardwareInterface>EffortJointInterface</hardwareInterface>
-        </joint>
-        <actuator name="motor2">
-            <hardwareInterface>EffortJointInterface</hardwareInterface>
-            <mechanicalReduction>1</mechanicalReduction>
-        </actuator>
+      <type>transmission_interface/SimpleTransmission</type>
+      <joint name="base_to_right_rear_wheel">
+        <hardwareInterface>EffortJointInterface</hardwareInterface>
+      </joint>
+      <actuator name="motor2">
+        <hardwareInterface>EffortJointInterface</hardwareInterface>
+        <mechanicalReduction>1</mechanicalReduction>
+      </actuator>
     </transmission>
 </robot>

Commit message: fix hokuyo3d showing and tf

File: third_robot_description/urdf/third_robot.xacro (robot description, xacro)
@@ -46,5 +46,5 @@
     <link name="front_top_3durg">
       <visual>
-        <origin rpy="0 0 0" xyz="0 0 0"/>
+        <origin rpy="0 0 0" xyz="-0.10 0 0"/>
         <geometry>
           <mesh filename="package://third_robot_description/meshes/3DURG/hokuyo3durg.dae"/>
@@ -56,5 +56,5 @@
       <parent link="base_link"/>
       <child link="front_top_3durg"/>
-      <origin rpy="3.14159 0 0" xyz="0.40 0 0.75"/>
+      <origin rpy="3.14159 0 0" xyz="0.50 0 0.75"/>
     </joint>
     <!-- front_bottom_lrf -->

Commit message: add merged_lrf frame

File: third_robot_description/urdf/third_robot.xacro (robot description, xacro)
@@ -153,4 +153,12 @@
       <origin rpy="0 0 0" xyz="0.45 0 0.72"/>
     </joint>
+    <joint name="base_to_merged_lrf" type="fixed">
+      <axis xyz="0 1 0"/>
+      <parent link="base_link" />
+      <child link="merged_lrf" />
+      <origin rpy="0 0 0" xyz="0 0 0.39"/>
+    </joint>
+    <link name="merged_lrf">
+    </link>
     <transmission name="tran1">
       <type>transmission_interface/SimpleTransmission</type>

Commit message: [WIP] gazebo用pointcloudプラグイン追加中

File: third_robot_description/urdf/third_robot.xacro (robot description, xacro)
@@ -1,4 +1,5 @@
 <?xml version="1.0"?>
 <robot name="origins" xmlns:xacro="http://www.ros.org/wiki/xacro">
+    <xacro:property name="M_PI" value="3.14159274"/>
     <xacro:property name="camera_link" value="0.05" /> <!-- Size of square 'camera' box -->
     <!-- Import all Gazebo-customization elements, including Gazebo colors -->
@@ -56,5 +57,6 @@
       <parent link="base_link"/>
       <child link="front_top_3durg"/>
-      <origin rpy="3.14159 0 0" xyz="0.40 0 0.75"/>
+      <origin rpy="${M_PI} 0 0" xyz="0.40 0 0.75"/>
+      <!--<origin rpy="3.14159 0 0" xyz="0.40 0 0.75"/>-->
     </joint>
     <!-- front_bottom_lrf -->

Commit message: [fix] gazebo用pointcloudプラグイン向き修正

File: third_robot_description/urdf/third_robot.xacro (robot description, xacro)
@@ -1,5 +1,4 @@
 <?xml version="1.0"?>
 <robot name="origins" xmlns:xacro="http://www.ros.org/wiki/xacro">
-    <xacro:property name="M_PI" value="3.14159274"/>
     <xacro:property name="camera_link" value="0.05" /> <!-- Size of square 'camera' box -->
     <!-- Import all Gazebo-customization elements, including Gazebo colors -->
@@ -57,5 +56,23 @@
       <parent link="base_link"/>
       <child link="front_top_3durg"/>
-      <origin rpy="${M_PI} 0 0" xyz="0.40 0 0.75"/>
+      <origin rpy="0 0 0" xyz="0.40 0 0.75"/>
+      <!-- <origin rpy="${M_PI} 0 0" xyz="0.40 0 0.75"/>-->
+      <!--<origin rpy="3.14159 0 0" xyz="0.40 0 0.75"/>-->
+    </joint>
+    <link name="front_top_3durg_rgbd_optical_frame">
+      <visual>
+        <origin rpy="0 0 0" xyz="0 0 0"/>
+        <geometry>
+          <mesh filename="package://third_robot_description/meshes/3DURG/hokuyo3durg.dae"/>
+        </geometry>
+      </visual>
+    </link>
+    <joint name="front_top_3durg_to_rgbd_optical_frame" type="fixed">
+      <axis xyz="0 1 0"/>
+      <parent link="front_top_3durg"/>
+      <child link="front_top_3durg_rgbd_optical_frame"/>
+      <origin rpy="${PI/2} ${PI} ${PI/2}"/>
+      <!-- <origin rpy="0 ${M_PI*0.5} 0" xyz="0.0 0.0 0.0"/> -->
+      <!-- <origin rpy="${M_PI} 0 0" xyz="0.40 0 0.75"/>-->
       <!--<origin rpy="3.14159 0 0" xyz="0.40 0 0.75"/>-->
     </joint>

Commit message: [fix] pointcloud用リンクの余分な要素を削除．

File: third_robot_description/urdf/third_robot.xacro (robot description, xacro)
@@ -60,12 +60,5 @@
       <!--<origin rpy="3.14159 0 0" xyz="0.40 0 0.75"/>-->
     </joint>
-    <link name="front_top_3durg_rgbd_optical_frame">
-      <visual>
-        <origin rpy="0 0 0" xyz="0 0 0"/>
-        <geometry>
-          <mesh filename="package://third_robot_description/meshes/3DURG/hokuyo3durg.dae"/>
-        </geometry>
-      </visual>
-    </link>
+    <link name="front_top_3durg_rgbd_optical_frame"/>
     <joint name="front_top_3durg_to_rgbd_optical_frame" type="fixed">
       <axis xyz="0 1 0"/>

Commit message: [fix] 仮想ステアリンクの余分なvisual要素を削除．

File: third_robot_description/urdf/third_robot.xacro (robot description, xacro)
@@ -86,12 +86,5 @@
     </joint>
     <!-- steer -->
-    <link name="steer">
-        <visual>
-            <origin rpy="0 0 0" xyz="0 0 0"/>
-            <geometry>
-                <mesh filename="package://third_robot_description/meshes/LRF/UTM-30LX.dae"/>
-            </geometry>
-        </visual>
-    </link>
+    <link name="steer"/>
     <joint name="base_to_steer" type="fixed">
         <axis xyz="0 1 0"/>

File: third_robot_description/urdf/third_robot_macro.xacro (robot description, xacro)
@@ -60,10 +60,4 @@
         <!-- steer_right -->
         <link name="steer_${right_left}">
-            <visual>
-                <origin rpy="0 0 0" xyz="0 0 0"/>
-                <geometry>
-                    <mesh filename="package://third_robot_description/meshes/LRF/UTM-30LX.dae"/>
-                </geometry>
-            </visual>
             <inertial>
                 <mass value="1.0" />

Commit message: [fix] 3Dセンサの向きを逆さに修正

File: third_robot_description/urdf/third_robot.xacro (robot description, xacro)
@@ -56,7 +56,5 @@
       <parent link="base_link"/>
       <child link="front_top_3durg"/>
-      <origin rpy="0 0 0" xyz="0.40 0 0.75"/>
-      <!-- <origin rpy="${M_PI} 0 0" xyz="0.40 0 0.75"/>-->
-      <!--<origin rpy="3.14159 0 0" xyz="0.40 0 0.75"/>-->
+      <origin rpy="${PI} 0 0" xyz="0.40 0 0.75"/>
     </joint>
     <link name="front_top_3durg_rgbd_optical_frame"/>
@@ -66,7 +64,4 @@
       <child link="front_top_3durg_rgbd_optical_frame"/>
       <origin rpy="${PI/2} ${PI} ${PI/2}"/>
-      <!-- <origin rpy="0 ${M_PI*0.5} 0" xyz="0.0 0.0 0.0"/> -->
-      <!-- <origin rpy="${M_PI} 0 0" xyz="0.40 0 0.75"/>-->
-      <!--<origin rpy="3.14159 0 0" xyz="0.40 0 0.75"/>-->
     </joint>
     <!-- front_bottom_lrf -->
