Commit message: [modify] steer joint の属性をrevoluteに修正．

File: third_robot_control/steer_drive_controller/test/wheel.xacro (robot description, xacro)
@@ -3,4 +3,6 @@
   <xacro:property name="steer_radius" value="0.05" /> <!-- Link 1 -->
   <xacro:property name="steer_thickness" value="0.02" /> <!-- Link 1 -->
+  <xacro:property name="steer_effort"   value="10.0"/>
+  <xacro:property name="steer_velocity" value="5.0"/>
   <macro name="front_wheel" params="name parent radius thickness length width axel_offset right_left steer_height *origin">
     <link name="${name}_steer_link">
@@ -23,5 +25,5 @@
       </collision>
     </link>
-    <joint name="${name}_steer_joint" type="continuous">
+    <joint name="${name}_steer_joint" type="revolute">
       <parent link="${parent}_link"/>
       <child link="${name}_steer_link"/>
@@ -29,5 +31,8 @@
       <!--insert_block name="origin"/-->
       <axis xyz="0 0 1"/>
-    </joint>
+      <limit effort="${steer_effort}"
+             lower="${-180.0 * deg_to_rad}" upper="${180.0 * deg_to_rad}"
+             velocity="${steer_velocity}"/>
+     </joint>
     <link name="${name}_link">
       <inertial>

Commit message: [modify] front wheel joint のlink名を修正．

File: third_robot_control/steer_drive_controller/test/wheel.xacro (robot description, xacro)
@@ -35,5 +35,5 @@
              velocity="${steer_velocity}"/>
      </joint>
-    <link name="${name}_link">
+    <link name="${name}_wheel_link">
       <inertial>
         <origin xyz="0 0 0" rpy="0 0 0"/>
@@ -56,5 +56,5 @@
     <joint name="${name}_joint" type="continuous">
       <parent link="${name}_steer_link"/>
-      <child link="${name}_link"/>
+      <child link="${name}_wheel_link"/>
       <origin xyz="0 0 ${-steer_height}" rpy="${-90 * deg_to_rad} 0 0"/>
       <axis xyz="0 0 1"/>
