Commit message: [modify] xacroで仮想Steer付きロボットモデルを作成

File: third_robot_control/steer_drive_controller/test/steerbot.xacro (robot description, xacro)
@@ -7,8 +7,10 @@
   <xacro:property name="deg_to_rad" value="0.01745329251994329577"/>
   <!-- Constants for robot dimensions -->
-  <xacro:property name="width" value="0.5" /> <!-- Square dimensions (widthxwidth) of beams -->
+  <xacro:property name="length" value="0.5" />
+  <xacro:property name="width" value="0.3" />
   <xacro:property name="wheel_radius" value="0.11" /> <!-- Link 1 -->
   <xacro:property name="thickness" value="0.086" /> <!-- Link 2 -->
   <xacro:property name="axel_offset" value="0.05" /> <!-- Space btw top of beam and the each joint -->
+  <xacro:property name="steer_offset" value="0.02" /> <!-- Link 1 -->
   <!-- Links: inertial,visual,collision -->
   <link name="base_link">
@@ -21,5 +23,5 @@
     <visual>
       <geometry>
-        <box size="${width} 0.1 0.1"/>
+        <box size="${length} ${width} 0.1"/>
       </geometry>
     </visual>
@@ -28,5 +30,5 @@
       <origin xyz="0 0 0"/>
       <geometry>
-        <box size="${width} 0.1 0.1"/>
+        <box size="${length} ${width} 0.1"/>
       </geometry>
     </collision>
@@ -51,10 +53,18 @@
   </joint>
   <!-- Wheels -->
-  <wheel name="wheel_0" parent="base" radius="${wheel_radius}" thickness="${thickness}">
-    <origin xyz="${width/2+axel_offset} 0 0" rpy="${-90 * deg_to_rad} 0 0"/>
-  </wheel>
-  <wheel name="wheel_1" parent="base" radius="${wheel_radius}" thickness="${thickness}">
-    <origin xyz="${-width/2+axel_offset} 0 0" rpy="${-90 * deg_to_rad} 0 0"/>
-  </wheel>
+  <front_wheel name="wheel_front_right" parent="base" radius="${wheel_radius}" thickness="${thickness}"
+      length="${length}" width="${width}" axel_offset="${axel_offset}" right_left="1" steer_height="${wheel_radius+steer_offset}">
+    <origin xyz="${length/2-axel_offset} ${width/2+axel_offset} 0" rpy="${-90 * deg_to_rad} 0 0"/>
+  </front_wheel>
+  <front_wheel name="wheel_front_left" parent="base" radius="${wheel_radius}" thickness="${thickness}"
+      length="${length}" width="${width}" axel_offset="${axel_offset}" right_left="-1" steer_height="${wheel_radius+steer_offset}">
+    <origin xyz="${length/2-axel_offset} ${-width/2-axel_offset} 0" rpy="${-90 * deg_to_rad} 0 0"/>
+  </front_wheel>
+  <rear_wheel name="wheel_rear_right" parent="base" radius="${wheel_radius}" thickness="${thickness}">
+    <origin xyz="${-length/2+axel_offset} ${width/2+axel_offset} 0" rpy="${-90 * deg_to_rad} 0 0"/>
+  </rear_wheel>
+  <rear_wheel name="wheel_rear_left" parent="base" radius="${wheel_radius}" thickness="${thickness}">
+    <origin xyz="${-length/2+axel_offset} ${-width/2-axel_offset} 0" rpy="${-90 * deg_to_rad} 0 0"/>
+  </rear_wheel>
   <!-- Colour -->
   <gazebo reference="base_link">

File: third_robot_control/steer_drive_controller/test/wheel.xacro (robot description, xacro)
@@ -1,5 +1,73 @@
 <?xml version="1.0"?>
 <robot xmlns:xacro="http://www.ros.org/wiki/xacro">
-  <macro name="wheel" params="name parent radius thickness *origin">
+  <xacro:property name="steer_radius" value="0.05" /> <!-- Link 1 -->
+  <xacro:property name="steer_thickness" value="0.02" /> <!-- Link 1 -->
+  <macro name="front_wheel" params="name parent radius thickness length width axel_offset right_left steer_height *origin">
+    <link name="${name}_steer_link">
+      <inertial>
+        <origin xyz="0 0 0" rpy="0 0 0"/>
+        <mass value="1"/>
+        <inertia ixx="0.2" ixy="0" ixz="0" iyy="0.2" iyz="0" izz="0.2"/>
+      </inertial>
+      <visual>
+        <origin xyz="0 0 0" rpy="0 0 0"/>
+        <geometry>
+          <cylinder radius="${steer_radius}" length="${steer_thickness}"/>
+        </geometry>
+      </visual>
+      <collision>
+        <origin xyz="0 0 0" rpy="0 0 0"/>
+        <geometry>
+          <cylinder radius="${steer_radius}" length="${steer_thickness}"/>
+        </geometry>
+      </collision>
+    </link>
+    <joint name="${name}_steer_joint" type="continuous">
+      <parent link="${parent}_link"/>
+      <child link="${name}_steer_link"/>
+      <origin xyz="${length/2-axel_offset} ${right_left*(width/2+axel_offset)} ${steer_height}" rpy="0 0 0"/>
+      <!--insert_block name="origin"/-->
+      <axis xyz="0 0 1"/>
+    </joint>
+    <link name="${name}_link">
+      <inertial>
+        <origin xyz="0 0 0" rpy="0 0 0"/>
+        <mass value="1"/>
+        <inertia ixx="0.2" ixy="0" ixz="0" iyy="0.2" iyz="0" izz="0.2"/>
+      </inertial>
+      <visual>
+        <origin xyz="0 0 0" rpy="0 0 0"/>
+        <geometry>
+          <cylinder radius="${wheel_radius}" length="${thickness}"/>
+        </geometry>
+      </visual>
+      <collision>
+        <origin xyz="0 0 0" rpy="0 0 0"/>
+        <geometry>
+          <cylinder radius="${wheel_radius}" length="${thickness}"/>
+        </geometry>
+      </collision>
+    </link>
+    <joint name="${name}_joint" type="continuous">
+      <parent link="${name}_steer_link"/>
+      <child link="${name}_link"/>
+      <origin xyz="0 0 ${-steer_height}" rpy="${-90 * deg_to_rad} 0 0"/>
+      <axis xyz="0 0 1"/>
+    </joint>
+    <!-- Transmission is important to link the joints and the controller -->
+    <transmission name="${name}_joint_trans" type="SimpleTransmission">
+      <actuator name="${name}_joint_motor"/>
+      <joint name="${name}_joint"/>
+      <mechanicalReduction>1</mechanicalReduction>
+      <motorTorqueConstant>1</motorTorqueConstant>
+    </transmission>
+    <gazebo reference="${name}_steer_link">
+      <material>Gazebo/Blue</material>
+    </gazebo>
+    <gazebo reference="${name}_link">
+      <material>Gazebo/Red</material>
+    </gazebo>
+  </macro>
+  <macro name="rear_wheel" params="name parent radius thickness *origin">
     <link name="${name}_link">
       <inertial>

Commit message: [add] rostest用steerbotを追加

File: third_robot_control/steer_drive_controller/test/steerbot.xacro (robot description, xacro)
@@ -53,16 +53,16 @@
   </joint>
   <!-- Wheels -->
-  <front_wheel name="wheel_front_right" parent="base" radius="${wheel_radius}" thickness="${thickness}"
+  <front_wheel name="front_right" parent="base" radius="${wheel_radius}" thickness="${thickness}"
       length="${length}" width="${width}" axel_offset="${axel_offset}" right_left="1" steer_height="${wheel_radius+steer_offset}">
     <origin xyz="${length/2-axel_offset} ${width/2+axel_offset} 0" rpy="${-90 * deg_to_rad} 0 0"/>
   </front_wheel>
-  <front_wheel name="wheel_front_left" parent="base" radius="${wheel_radius}" thickness="${thickness}"
+  <front_wheel name="front_left" parent="base" radius="${wheel_radius}" thickness="${thickness}"
       length="${length}" width="${width}" axel_offset="${axel_offset}" right_left="-1" steer_height="${wheel_radius+steer_offset}">
     <origin xyz="${length/2-axel_offset} ${-width/2-axel_offset} 0" rpy="${-90 * deg_to_rad} 0 0"/>
   </front_wheel>
-  <rear_wheel name="wheel_rear_right" parent="base" radius="${wheel_radius}" thickness="${thickness}">
+  <rear_wheel name="rear_right" parent="base" radius="${wheel_radius}" thickness="${thickness}">
     <origin xyz="${-length/2+axel_offset} ${width/2+axel_offset} 0" rpy="${-90 * deg_to_rad} 0 0"/>
   </rear_wheel>
-  <rear_wheel name="wheel_rear_left" parent="base" radius="${wheel_radius}" thickness="${thickness}">
+  <rear_wheel name="rear_left" parent="base" radius="${wheel_radius}" thickness="${thickness}">
     <origin xyz="${-length/2+axel_offset} ${-width/2-axel_offset} 0" rpy="${-90 * deg_to_rad} 0 0"/>
   </rear_wheel>

File: third_robot_control/steer_drive_controller/test/wheel.xacro (robot description, xacro)
@@ -54,5 +54,5 @@
       </collision>
     </link>
-    <joint name="${name}_joint" type="continuous">
+    <joint name="${name}_wheel_joint" type="continuous">
       <parent link="${name}_steer_link"/>
       <child link="${name}_wheel_link"/>
@@ -61,7 +61,13 @@
     </joint>
     <!-- Transmission is important to link the joints and the controller -->
-    <transmission name="${name}_joint_trans" type="SimpleTransmission">
-      <actuator name="${name}_joint_motor"/>
-      <joint name="${name}_joint"/>
+    <transmission name="${name}_steer_joint_trans" type="SimpleTransmission">
+      <actuator name="${name}_steer_joint_motor"/>
+      <joint name="${name}_steer_joint"/>
+      <mechanicalReduction>1</mechanicalReduction>
+      <motorTorqueConstant>1</motorTorqueConstant>
+    </transmission>
+    <transmission name="${name}_wheel_joint_trans" type="SimpleTransmission">
+      <actuator name="${name}_wheel_joint_motor"/>
+      <joint name="${name}_wheel_joint"/>
       <mechanicalReduction>1</mechanicalReduction>
       <motorTorqueConstant>1</motorTorqueConstant>
@@ -70,10 +76,10 @@
       <material>Gazebo/Blue</material>
     </gazebo>
-    <gazebo reference="${name}_link">
+    <gazebo reference="${name}_wheel_link">
       <material>Gazebo/Red</material>
     </gazebo>
   </macro>
   <macro name="rear_wheel" params="name parent radius thickness *origin">
-    <link name="${name}_link">
+    <link name="${name}_wheel_link">
       <inertial>
         <origin xyz="0 0 0" rpy="0 0 0"/>
@@ -94,18 +100,18 @@
       </collision>
     </link>
-    <joint name="${name}_joint" type="continuous">
+    <joint name="${name}_wheel_joint" type="continuous">
       <parent link="${parent}_link"/>
-      <child link="${name}_link"/>
+      <child link="${name}_wheel_link"/>
       <insert_block name="origin"/>
       <axis xyz="0 0 1"/>
     </joint>
     <!-- Transmission is important to link the joints and the controller -->
-    <transmission name="${name}_joint_trans" type="SimpleTransmission">
-      <actuator name="${name}_joint_motor"/>
-      <joint name="${name}_joint"/>
+    <transmission name="${name}_wheel_joint_trans" type="SimpleTransmission">
+      <actuator name="${name}_wheel_joint_motor"/>
+      <joint name="${name}_wheel_joint"/>
       <mechanicalReduction>1</mechanicalReduction>
       <motorTorqueConstant>1</motorTorqueConstant>
     </transmission>
-    <gazebo reference="${name}_link">
+    <gazebo reference="${name}_wheel_link">
       <material>Gazebo/Red</material>
     </gazebo>
